Commit message: Converted to using xacro for the model, added xacro to iris-ap launch file

File: simulator/vehicles/iris-ap/models/gimbal_small_2d/model.sdf.xacro (robot description, xacro)
@@ -1,5 +1,10 @@
 <?xml version='1.0'?>
-<sdf version='1.6'>
-  <model name='gimbal_small_2d'>
+<sdf version='1.6' xmlns:xacro="http://www.ros.org/wiki/xacro">
+  <xacro:property name="ros_namespace" value="$(arg ros_namespace)" />
+  <xacro:property name="camera_name" value="$(arg camera_name)" />
+  <xacro:property name="camera_width" value="$(arg camera_width)" />
+  <xacro:property name="camera_height" value="$(arg camera_height)" />
+  <xacro:property name="gimbal_initial_angle" value="$(arg gimbal_initial_angle)" />
+    <model name='gimbal_small_2d'>
     <pose>0 0 0.18 0 0 0</pose>
     <link name='base_link'>
@@ -128,6 +133,6 @@
           <horizontal_fov>2.0</horizontal_fov>
           <image>
-            <width>640</width>
-            <height>480</height>
+            <width>${camera_width}</width>
+            <height>${camera_height}</height>
           </image>
           <clip>
@@ -148,9 +153,9 @@
         <plugin name="camera_controller" filename="libgazebo_ros_camera.so">
           <ros>
-            <namespace>vehicle_1</namespace>
+            <namespace>${ros_namespace}</namespace>
             <!-- <argument>image_raw:=custom</argument> -->
             <!-- <argument>camera_info:=custom_info</argument> -->
           </ros>
-          <camera_name>camera</camera_name>
+          <camera_name>${camera_name}</camera_name>
           <frame_name>camera_link</frame_name>
           <hack_baseline>0.07</hack_baseline>
@@ -183,7 +188,8 @@
     <plugin name="gimbal_small_2d" filename="libGimbal2dPlugin.so">
       <ros>
-        <namespace>vehicle_1</namespace>
+        <namespace>${ros_namespace}</namespace>
       </ros>
       <joint>tilt_joint</joint>
+      <initial_angle>${gimbal_initial_angle}</initial_angle>
     </plugin>
   </model>

Commit message: Moved things around in iris-ap!

File: simulator/vehicles/iris-ap/models/gimbal_small_2d/model.sdf.xacro (robot description, xacro)
@@ -6,4 +6,5 @@
   <xacro:property name="camera_height" value="$(arg camera_height)" />
   <xacro:property name="gimbal_initial_angle" value="$(arg gimbal_initial_angle)" />
+  <xacro:property name="gimbal_meshes_directory" value="$(arg gimbal_meshes_directory)" />
     <model name='gimbal_small_2d'>
     <pose>0 0 0.18 0 0 0</pose>
@@ -24,5 +25,5 @@
          <mesh>
            <scale>0.001 0.001 0.001</scale>
-           <uri>model://gimbal_small_2d/meshes/base_main.dae</uri>
+           <uri>model:/${gimbal_meshes_directory}/base_main.dae</uri>
          </mesh>
         </geometry>
@@ -38,5 +39,5 @@
          <mesh>
            <scale>0.001 0.001 0.001</scale>
-           <uri>model://gimbal_small_2d/meshes/base_arm.dae</uri>
+           <uri>model://${gimbal_meshes_directory}/base_arm.dae</uri>
          </mesh>
         </geometry>
@@ -85,5 +86,5 @@
          <mesh>
            <scale>0.001 0.001 0.001</scale>
-           <uri>model://gimbal_small_2d/meshes/tilt.dae</uri>
+           <uri>model://${gimbal_meshes_directory}/tilt.dae</uri>
          </mesh>
         </geometry>
@@ -100,5 +101,5 @@
          <mesh>
            <scale>0.001 0.001 0.001</scale>
-           <uri>model://gimbal_small_2d/meshes/tilt.dae</uri>
+           <uri>model://${gimbal_meshes_directory}/tilt.dae</uri>
          </mesh>
         </geometry>
