Commit message: Use xacro:parameter with  fixes loading issue

File: simulator/vehicles/iris-ap/models/iris_ap/model.sdf.xacro (robot description, xacro)
@@ -1,6 +1,8 @@
 <?xml version='1.0'?>
 <sdf version="1.6" xmlns:xacro='http://ros.org/wiki/xacro'>
-  <xacro:arg name="fdm_addr" default="127.0.0.1"/>
-  <xacro:arg name="listen_addr" default="127.0.0.1"/>
+  <!-- <xacro:arg name="fdm_addr" default="127.0.0.1"/> -->
+  <!-- <xacro:arg name="listen_addr" default="127.0.0.1"/> -->
+  <xacro:property name="fdm_addr" value="$(arg fdm_addr)"/>
+  <xacro:property name="listen_addr" value="$(arg listen_addr)"/>
   <model name="iris_demo">
     <include>
@@ -23,358 +25,4 @@
       </axis>
     </joint>
-    <!-- visual markers for debugging
-    <link name="rotor_0_blade_1_cp">
-      <gravity>0</gravity>
-      <pose>0.13 -0.22 0.216 0 -0 0</pose>
-      <visual name='rotor_0_visual_root'>
-        <pose>0 0 0 0 -0 0</pose>
-        <geometry>
-          <sphere>
-            <radius>0.01</radius>
-          </sphere>
-        </geometry>
-      </visual>
-      <visual name='rotor_0_visual_tip'>
-        <pose>0.12 0 0 0 -0 0</pose>
-        <geometry>
-          <sphere>
-            <radius>0.01</radius>
-          </sphere>
-        </geometry>
-      </visual>
-      <visual name='rotor_0_visual_cp'>
-        <pose>0.084 0 0 0 -0 0</pose>
-        <geometry>
-          <sphere>
-            <radius>0.003</radius>
-          </sphere>
-        </geometry>
-      </visual>
-      <visual name='rotor_0_visual_cp_forward'>
-        <pose>0.084 0.02 0 0 -0 0</pose>
-        <geometry>
-          <sphere>
-            <radius>0.003</radius>
-          </sphere>
-        </geometry>
-      </visual>
-      <visual name='rotor_0_visual_cp_upward'>
-        <pose>0.084 0 0.02 0 -0 0</pose>
-        <geometry>
-          <sphere>
-            <radius>0.003</radius>
-          </sphere>
-        </geometry>
-      </visual>
-    </link>
-    <link name="rotor_0_blade_2_cp">
-      <gravity>0</gravity>
-      <pose>0.13 -0.22 0.216 0 -0 0</pose>
-      <visual name='rotor_0_visual_root'>
-        <pose>0 0 0 0 -0 0</pose>
-        <geometry>
-          <sphere>
-            <radius>0.01</radius>
-          </sphere>
-        </geometry>
-      </visual>
-      <visual name='rotor_0_visual_tip'>
-        <pose>-0.12 0 0 0 -0 0</pose>
-        <geometry>
-          <sphere>
-            <radius>0.01</radius>
-          </sphere>
-        </geometry>
-      </visual>
-      <visual name='rotor_0_visual_cp'>
-        <pose>-0.084 0 0 0 -0 0</pose>
-        <geometry>
-          <sphere>
-            <radius>0.003</radius>
-          </sphere>
-        </geometry>
-      </visual>
-      <visual name='rotor_0_visual_cp_forward'>
-        <pose>-0.084 -0.02 0 0 -0 0</pose>
-        <geometry>
-          <sphere>
-            <radius>0.003</radius>
-          </sphere>
-        </geometry>
-      </visual>
-      <visual name='rotor_0_visual_cp_upward'>
-        <pose>-0.084 0 0.02 0 -0 0</pose>
-        <geometry>
-          <sphere>
-            <radius>0.003</radius>
-          </sphere>
-        </geometry>
-      </visual>
-    </link>
-    <link name="rotor_1_blade_1_cp">
-      <gravity>0</gravity>
-      <pose>-0.13 0.2 0.216 0 -0 0</pose>
-      <visual name='rotor_1_visual_root'>
-        <pose>0 0 0 0 -0 0</pose>
-        <geometry>
-          <sphere>
-            <radius>0.01</radius>
-          </sphere>
-        </geometry>
-      </visual>
-      <visual name='rotor_1_visual_tip'>
-        <pose>0.12 0 0 0 -0 0</pose>
-        <geometry>
-          <sphere>
-            <radius>0.01</radius>
-          </sphere>
-        </geometry>
-      </visual>
-      <visual name='rotor_1_visual_cp'>
-        <pose>0.084 0 0 0 -0 0</pose>
-        <geometry>
-          <sphere>
-            <radius>0.003</radius>
-          </sphere>
-        </geometry>
-      </visual>
-      <visual name='rotor_1_visual_cp_forward'>
-        <pose>0.084 0.02 0 0 -0 0</pose>
-        <geometry>
-          <sphere>
-            <radius>0.003</radius>
-          </sphere>
-        </geometry>
-      </visual>
-      <visual name='rotor_1_visual_cp_upward'>
-        <pose>0.084 0 0.02 0 -0 0</pose>
-        <geometry>
-          <sphere>
-            <radius>0.003</radius>
-          </sphere>
-        </geometry>
-      </visual>
-    </link>
-    <link name="rotor_1_blade_2_cp">
-      <gravity>0</gravity>
-      <pose>-0.13 0.2 0.216 0 -0 0</pose>
-      <visual name='rotor_1_visual_root'>
-        <pose>0 0 0 0 -0 0</pose>
-        <geometry>
-          <sphere>
-            <radius>0.01</radius>
-          </sphere>
-        </geometry>
-      </visual>
-      <visual name='rotor_1_visual_tip'>
-        <pose>-0.12 0 0 0 -0 0</pose>
-        <geometry>
-          <sphere>
-            <radius>0.01</radius>
-          </sphere>
-        </geometry>
-      </visual>
-      <visual name='rotor_1_visual_cp'>
-        <pose>-0.084 0 0 0 -0 0</pose>
-        <geometry>
-          <sphere>
-            <radius>0.003</radius>
-          </sphere>
-        </geometry>
-      </visual>
-      <visual name='rotor_1_visual_cp_forward'>
-        <pose>-0.084 -0.02 0 0 -0 0</pose>
-        <geometry>
-          <sphere>
-            <radius>0.003</radius>
-          </sphere>
-        </geometry>
-      </visual>
-      <visual name='rotor_1_visual_cp_upward'>
-        <pose>-0.084 0 0.02 0 -0 0</pose>
-        <geometry>
-          <sphere>
-            <radius>0.003</radius>
-          </sphere>
-        </geometry>
-      </visual>
-    </link>
-    <link name="rotor_2_blade_1_cp">
-      <gravity>0</gravity>
-      <pose>0.13 0.22 0.216 0 -0 0</pose>
-      <visual name='rotor_2_visual_root'>
-        <pose>0 0 0 0 -0 0</pose>
-        <geometry>
-          <sphere>
-            <radius>0.01</radius>
-          </sphere>
-        </geometry>
-      </visual>
-      <visual name='rotor_2_visual_tip'>
-        <pose>0.12 0 0 0 -0 0</pose>
-        <geometry>
-          <sphere>
-            <radius>0.01</radius>
-          </sphere>
-        </geometry>
-      </visual>
-      <visual name='rotor_2_visual_cp'>
-        <pose>0.084 0 0 0 -0 0</pose>
-        <geometry>
-          <sphere>
-            <radius>0.003</radius>
-          </sphere>
-        </geometry>
-      </visual>
-      <visual name='rotor_2_visual_cp_forward'>
-        <pose>0.084 -0.02 0 0 -0 0</pose>
-        <geometry>
-          <sphere>
-            <radius>0.003</radius>
-          </sphere>
-        </geometry>
-      </visual>
-      <visual name='rotor_2_visual_cp_upward'>
-        <pose>0.084 0 0.02 0 -0 0</pose>
-        <geometry>
-          <sphere>
-            <radius>0.003</radius>
-          </sphere>
-        </geometry>
-      </visual>
-    </link>
-    <link name="rotor_2_blade_2_cp">
-      <gravity>0</gravity>
-      <pose>0.13 0.22 0.216 0 -0 0</pose>
-      <visual name='rotor_2_visual_root'>
-        <pose>0 0 0 0 -0 0</pose>
-        <geometry>
-          <sphere>
-            <radius>0.01</radius>
-          </sphere>
-        </geometry>
-      </visual>
-      <visual name='rotor_2_visual_tip'>
-        <pose>-0.12 0 0 0 -0 0</pose>
-        <geometry>
-          <sphere>
-            <radius>0.01</radius>
-          </sphere>
-        </geometry>
-      </visual>
-      <visual name='rotor_2_visual_cp'>
-        <pose>-0.084 0 0 0 -0 0</pose>
-        <geometry>
-          <sphere>
-            <radius>0.003</radius>
-          </sphere>
-        </geometry>
-      </visual>
-      <visual name='rotor_2_visual_cp_forward'>
-        <pose>-0.084 0.02 0 0 -0 0</pose>
-        <geometry>
-          <sphere>
-            <radius>0.003</radius>
-          </sphere>
-        </geometry>
-      </visual>
-      <visual name='rotor_2_visual_cp_upward'>
-        <pose>-0.084 0 0.02 0 -0 0</pose>
-        <geometry>
-          <sphere>
-            <radius>0.003</radius>
-          </sphere>
-        </geometry>
-      </visual>
-    </link>
-    <link name="rotor_3_blade_1_cp">
-      <gravity>0</gravity>
-      <pose>-0.13 -0.2 0.216 0 -0 0</pose>
-      <visual name='rotor_3_visual_root'>
-        <pose>0 0 0 0 -0 0</pose>
-        <geometry>
-          <sphere>
-            <radius>0.01</radius>
-          </sphere>
-        </geometry>
-      </visual>
-      <visual name='rotor_3_visual_tip'>
-        <pose>0.12 0 0 0 -0 0</pose>
-        <geometry>
-          <sphere>
-            <radius>0.01</radius>
-          </sphere>
-        </geometry>
-      </visual>
-      <visual name='rotor_3_visual_cp'>
-        <pose>0.084 0 0 0 -0 0</pose>
-        <geometry>
-          <sphere>
-            <radius>0.003</radius>
-          </sphere>
-        </geometry>
-      </visual>
-      <visual name='rotor_3_visual_cp_forward'>
-        <pose>0.084 -0.02 0 0 -0 0</pose>
-        <geometry>
-          <sphere>
-            <radius>0.003</radius>
-          </sphere>
-        </geometry>
-      </visual>
-      <visual name='rotor_3_visual_cp_upward'>
-        <pose>0.084 0 0.02 0 -0 0</pose>
-        <geometry>
-          <sphere>
-            <radius>0.003</radius>
-          </sphere>
-        </geometry>
-      </visual>
-    </link>
-    <link name="rotor_3_blade_2_cp">
-      <gravity>0</gravity>
-      <pose>-0.13 -0.2 0.216 0 -0 0</pose>
-      <visual name='rotor_3_visual_root'>
-        <pose>0 0 0 0 -0 0</pose>
-        <geometry>
-          <sphere>
-            <radius>0.01</radius>
-          </sphere>
-        </geometry>
-      </visual>
-      <visual name='rotor_3_visual_tip'>
-        <pose>-0.12 0 0 0 -0 0</pose>
-        <geometry>
-          <sphere>
-            <radius>0.01</radius>
-          </sphere>
-        </geometry>
-      </visual>
-      <visual name='rotor_3_visual_cp'>
-        <pose>-0.084 0 0 0 -0 0</pose>
-        <geometry>
-          <sphere>
-            <radius>0.003</radius>
-          </sphere>
-        </geometry>
-      </visual>
-      <visual name='rotor_3_visual_cp_forward'>
-        <pose>-0.084 0.02 0 0 -0 0</pose>
-        <geometry>
-          <sphere>
-            <radius>0.003</radius>
-          </sphere>
-        </geometry>
-      </visual>
-      <visual name='rotor_3_visual_cp_upward'>
-        <pose>-0.084 0 0.02 0 -0 0</pose>
-        <geometry>
-          <sphere>
-            <radius>0.003</radius>
-          </sphere>
-        </geometry>
-      </visual>
-    </link>
-    -->
     <!-- plugins -->
     <plugin name="rotor_0_blade_1" filename="libLiftDragPlugin.so">
@@ -507,6 +155,6 @@
     </plugin>
     <plugin name="arducopter_plugin" filename="libArduPilotPlugin.so">
-      <fdm_addr>$(arg fdm_addr)</fdm_addr>
-      <listen_addr>$(arg listen_addr)</listen_addr>
+      <fdm_addr>${fdm_addr}</fdm_addr>
+      <listen_addr>${listen_addr}</listen_addr>
       <fdm_port_in>9002</fdm_port_in>
       <fdm_port_out>9003</fdm_port_out>

Commit message: Added rangefinder into iris-ap model

File: simulator/vehicles/iris-ap/models/iris_ap/model.sdf.xacro (robot description, xacro)
@@ -3,4 +3,5 @@
   <!-- <xacro:arg name="fdm_addr" default="127.0.0.1"/> -->
   <!-- <xacro:arg name="listen_addr" default="127.0.0.1"/> -->
+  <xacro:property name="ros_namespace" value="$(arg ros_namespace)"/>
   <xacro:property name="fdm_addr" value="$(arg fdm_addr)"/>
   <xacro:property name="listen_addr" value="$(arg listen_addr)"/>
@@ -25,4 +26,61 @@
       </axis>
     </joint>
+    <link name="hokuyo_link">
+      <!-- Visuals / Collisions omitted for this example -->
+      <sensor type="gpu_ray" name="head_hokuyo_sensor">
+        <ray>
+          <scan>
+            <horizontal>
+              <samples>10</samples>
+              <resolution>1</resolution>
+              <min_angle>-0.087</min_angle>
+              <max_angle>0.087</max_angle>
+            </horizontal>
+            <vertical>
+              <samples>10</samples>
+              <resolution>1</resolution>
+              <min_angle>-0.087</min_angle>
+              <max_angle>0.087</max_angle>
+            </vertical>
+          </scan>
+          <range>
+            <min>0.10</min>
+            <max>10.0</max>
+            <resolution>0.01</resolution>
+          </range>
+          <!-- Using gazebo's noise instead of plugin's -->
+          <noise>
+            <type>gaussian</type>
+            <mean>0.0</mean>
+            <stddev>0.01</stddev>
+          </noise>
+        </ray>
+        <!-- Using gazebo's update rate instead of plugin's -->
+        <update_rate>30</update_rate>
+        <plugin name="laser" filename="libgazebo_ros_ray_sensor.so">
+          <!-- Change namespace and output topic so published topic is /rrbot/laser/scan -->
+          <ros>
+            <namespace>${ros_namespace}</namespace>
+          </ros>
+          <!-- Set output to sensor_msgs/LaserScan to get same output type as gazebo_ros_laser -->
+          <output_type>sensor_msgs/Range</output_type>
+          <!-- <frame_name> ommited, will default to hokuo_link -->
+          <radiation_type>infrared</radiation_type>
+        </plugin>
+      </sensor>
+    </link>
+    <joint name="iris_hokuyo_mount" type="revolute">
+      <parent>iris::base_link</parent>
+      <child>hokuyo_link</child>
+      <axis>
+        <limit>
+          <lower>0</lower>
+          <upper>0</upper>
+        </limit>
+        <xyz>-1 0 1</xyz>
+        <rpy>0 0.0 0</rpy>
+        <use_parent_model_frame>true</use_parent_model_frame>
+      </axis>
+    </joint>
     <!-- plugins -->
     <plugin name="rotor_0_blade_1" filename="libLiftDragPlugin.so">

Commit message: Continued trying to adjust the rangefinder so pointing in the correct direction

File: simulator/vehicles/iris-ap/models/iris_ap/model.sdf.xacro (robot description, xacro)
@@ -27,4 +27,13 @@
     </joint>
     <link name="hokuyo_link">
+      <pose>-0.5 0 -1 0 -1.57075 0</pose>
+      <!-- <visual name="my_visual">
+          <pose>0 0 0 0 0</pose>
+          <geometry>
+            <box>
+              <size>1.0 0.1 0.1</size>
+            </box>
+          </geometry>
+      </visual> -->
       <!-- Visuals / Collisions omitted for this example -->
       <sensor type="gpu_ray" name="head_hokuyo_sensor">
@@ -70,8 +79,8 @@
       </sensor>
     </link>
-    <joint name="iris_hokuyo_mount" type="revolute">
+    <joint name="iris_hokuyo_mount" type="fixed">
       <parent>iris::base_link</parent>
       <child>hokuyo_link</child>
-      <axis>
+      <!-- <axis>
         <limit>
           <lower>0</lower>
@@ -81,5 +90,5 @@
         <rpy>0 0.0 0</rpy>
         <use_parent_model_frame>true</use_parent_model_frame>
-      </axis>
+      </axis> -->
     </joint>
     <!-- plugins -->

Commit message: Removed inertia and mass from sensor and set min/max resolution

File: simulator/vehicles/iris-ap/models/iris_ap/model.sdf.xacro (robot description, xacro)
@@ -27,13 +27,17 @@
     </joint>
     <link name="hokuyo_link">
-      <pose>-0.5 0 -1 0 -1.57075 0</pose>
-      <!-- <visual name="my_visual">
-          <pose>0 0 0 0 0</pose>
-          <geometry>
-            <box>
-              <size>1.0 0.1 0.1</size>
-            </box>
-          </geometry>
-      </visual> -->
+      <pose>0 0 0 0 1.57075 0</pose>
+      <inertial>
+        <mass>0.016</mass>
+        <inertia>
+          <ixx>0.0001</ixx>
+          <ixy>0</ixy>
+          <ixz>0</ixz>
+          <iyy>0.0001</iyy>
+          <iyz>0</iyz>
+          <izz>0.0001</izz>
+        <!-- low intertia necessary to avoid to disturb the drone -->
+        </inertia>
+      </inertial>
       <!-- Visuals / Collisions omitted for this example -->
       <sensor type="gpu_ray" name="head_hokuyo_sensor">
@@ -54,6 +58,6 @@
           </scan>
           <range>
-            <min>0.10</min>
-            <max>10.0</max>
+            <min>0.01</min>
+            <max>20.0</max>
             <resolution>0.01</resolution>
           </range>
